File: GhettoTMC.kicad_pcb (KiCad board)
At the start: 2 copper layers, 48 parts, among them J1 Stepper_X, J10 Board Z, J11 Board E, J2 Stepper_Y, J3 Stepper_Z1, J4 Stepper_Z2, J5 Stepper_E, J6 Data, J7 POWER IN, J8 Board X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

Commit message: PCB work
Parts:
- added M1: MountingHole_3.2mm_M3, MountingHole:MountingHole_3.2mm_M3, F.Cu at (166.4, 143.5)
- added M2: MountingHole_3.2mm_M3, MountingHole:MountingHole_3.2mm_M3, F.Cu at (166.4, 80.0)
Other:
- board outline added: 100.3 x 71.1 mm
- board text added: "GhettoTMC_SPR3.0 TMC2209"

Commit message: 24V net manual clearance
Routing:
- net +24V: track 190.6 -> 192.9 mm
- net GND: track 272.6 -> 270.5 mm
Other:
- board text added: "GhettoTMC_SPR3 TMC2209"
- board text removed: "GhettoTMC_SPR3.0 TMC2209"
Changed lines of the file:
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@@
     (thickness 1.6)
     (drawings 9)
-    (tracks 318)
+    (tracks 317)
     (zones 0)
     (modules 50)
@@
   )
   (setup
-    (last_trace_width 0.25)
+    (last_trace_width 1.5)
     (user_trace_width 0.5)
     (user_trace_width 1)
@@
     (visible_elements 7FFFFFFF)
     (pcbplotparams
-      (layerselection 0x010fc_ffffffff)
+      (layerselection 0x010f0_ffffffff)
       (usegerberextensions false)
       (usegerberattributes false)
@@
       (creategerberjobfile false)
       (excludeedgelayer true)
-      (linewidth 0.100000)
+      (linewidth 0.150000)
       (plotframeref false)
       (viasonmask false)
@@
       (outputformat 1)
       (mirror false)
-      (drillshape 1)
+      (drillshape 0)
       (scaleselection 1)
-      (outputdirectory ""))
+      (outputdirectory "Gerber/"))
   )
   (net 0 "")
@@
     )
   )
-  (gr_text "GhettoTMC_SPR3.0\nTMC2209" (at 122.555 101.6) (layer F.SilkS)
+  (gr_text "GhettoTMC_SPR3\nTMC2209" (at 122.555 101.6) (layer F.SilkS)
     (effects (font (size 2 2) (thickness 0.5) italic))
   )
@@
   (segment (start 85.645 118.11) (end 83.74 120.015) (width 1) (layer B.Cu) (net 2))
   (segment (start 92.71 118.11) (end 85.645 118.11) (width 1) (layer B.Cu) (net 2))
-  (segment (start 83.74 120.015) (end 83.74 123.19) (width 1) (layer B.Cu) (net 2))
   (segment (start 84.375 102.87) (end 83.74 103.505) (width 1) (layer B.Cu) (net 2))
   (segment (start 92.71 102.87) (end 84.375 102.87) (width 1) (layer B.Cu) (net 2))
@@
   (segment (start 105.41 115.57) (end 111.125 121.285) (width 1) (layer B.Cu) (net 2))
   (segment (start 126.365 122.555) (end 126.365 109.855) (width 1) (layer F.Cu) (net 2))
-  (via (at 142.24 121.92) (size 0.8) (drill 0.4) (layers F.Cu B.Cu) (net 2))
-  (segment (start 148.59 125.73) (end 146.05 125.73) (width 1) (layer F.Cu) (net 2))
-  (segment (start 146.05 125.73) (end 142.24 121.92) (width 1) (layer F.Cu) (net 2))
+  (via (at 143.51 120.65) (size 0.8) (drill 0.4) (layers F.Cu B.Cu) (net 2))
+  (segment (start 148.59 125.73) (end 143.51 120.65) (width 1) (layer F.Cu) (net 2))
   (segment (start 137.02137 125.73) (end 135.89 125.73) (width 1) (layer B.Cu) (net 2))
-  (segment (start 142.24 122.573518) (end 139.083518 125.73) (width 1) (layer B.Cu) (net 2))
   (segment (start 139.083518 125.73) (end 137.02137 125.73) (width 1) (layer B.Cu) (net 2))
-  (segment (start 142.24 121.92) (end 142.24 122.573518) (width 1) (layer B.Cu) (net 2))
+  (segment (start 143.51 121.303518) (end 139.083518 125.73) (width 1) (layer B.Cu) (net 2))
+  (segment (start 143.51 120.65) (end 143.51 121.303518) (width 1) (layer B.Cu) (net 2))
   (segment (start 153.67 130.81) (end 156.21 130.81) (width 1) (layer F.Cu) (net 3))
   (segment (start 156.21 130.81) (end 157.412081 130.81) (width 1) (layer F.Cu) (net 3))
@@
   (segment (start 153.67 115.57) (end 145.415 123.825) (width 0.5) (layer B.Cu) (net 22))
   (segment (start 145.415 123.825) (end 135.89 133.35) (width 0.5) (layer B.Cu) (net 22))
-  (segment (start 90.54 120.65) (end 91.57863 120.65) (width 1.5) (layer B.Cu) (net 23))
-  (segment (start 73.66 137.53) (end 90.54 120.65) (width 1.5) (layer B.Cu) (net 23))
-  (segment (start 91.57863 120.65) (end 92.71 120.65) (width 1.5) (layer B.Cu) (net 23))
   (segment (start 73.66 138.43) (end 73.66 137.53) (width 1.5) (layer B.Cu) (net 23))
   (segment (start 73.66 138.43) (end 73.66 139.33) (width 1.5) (layer B.Cu) (net 23))
-  (segment (start 157.554003 118.899999) (end 152.880001 118.899999) (width 1.5) (layer B.Cu) (net 23))
-  (segment (start 163.590001 112.864001) (end 157.554003 118.899999) (width 1.5) (layer B.Cu) (net 23))
-  (segment (start 163.590001 110.655999) (end 163.590001 112.864001) (width 1.5) (layer B.Cu) (net 23))
-  (segment (start 149.389999 122.390001) (end 148.59 123.19) (width 1.5) (layer B.Cu) (net 23))
-  (segment (start 153.744003 100.810001) (end 163.590001 110.655999) (width 1.5) (layer B.Cu) (net 23))
-  (segment (start 145.260001 100.810001) (end 153.744003 100.810001) (width 1.5) (layer B.Cu) (net 23))
-  (segment (start 152.880001 118.899999) (end 149.389999 122.390001) (width 1.5) (layer B.Cu) (net 23))
-  (segment (start 143.51 99.06) (end 145.260001 100.810001) (width 1.5) (layer B.Cu) (net 23))
   (segment (start 73.66 141.73) (end 73.66 138.43) (width 1.5) (layer B.Cu) (net 23))
   (segment (start 75.44 143.51) (end 73.66 141.73) (width 1.5) (layer B.Cu) (net 23))
@@
   (segment (start 144.78 127) (end 148.59 123.19) (width 1.5) (layer B.Cu) (net 23))
   (segment (start 144.78 135.89) (end 144.78 127) (width 1.5) (layer B.Cu) (net 23))
+  (segment (start 149.389999 122.390001) (end 148.59 123.19) (width 1.5) (layer B.Cu) (net 23))
+  (segment (start 152.880001 118.899999) (end 149.389999 122.390001) (width 1.5) (layer B.Cu) (net 23))
+  (segment (start 157.554003 118.899999) (end 152.880001 118.899999) (width 1.5) (layer B.Cu) (net 23))
+  (segment (start 143.51 99.06) (end 151.13 106.68) (width 1.5) (layer B.Cu) (net 23))
+  (segment (start 159.614002 106.68) (end 163.590001 110.655999) (width 1.5) (layer B.Cu) (net 23))
+  (segment (start 163.590001 110.655999) (end 163.590001 112.864001) (width 1.5) (layer B.Cu) (net 23))
+  (segment (start 151.13 106.68) (end 159.614002 106.68) (width 1.5) (layer B.Cu) (net 23))
+  (segment (start 163.590001 112.864001) (end 157.554003 118.899999) (width 1.5) (layer B.Cu) (net 23))
+  (segment (start 73.66 135.13) (end 81.79 127) (width 1.5) (layer B.Cu) (net 23))
+  (segment (start 73.66 138.43) (end 73.66 135.13) (width 1.5) (layer B.Cu) (net 23))
+  (segment (start 86.36 127) (end 92.71 120.65) (width 1.5) (layer B.Cu) (net 23))
+  (segment (start 81.79 127) (end 86.36 127) (width 1.5) (layer B.Cu) (net 23))
   (segment (start 139.680001 111.025001) (end 118.825 90.17) (width 0.5) (layer B.Cu) (net 24))
   (segment (start 118.825 90.17) (end 117.475 90.17) (width 0.5) (layer B.Cu) (net 24))
